File: PlacasPractica.sch (KiCad schematic (older format))
At the start: 66 parts, among them J1 USB_OTG, J2 Conn_01x10, J3 Conn_01x10, J4 CONN_02X05, SW1 SW_Push, U1 SAMD20J18A-AU, U2 XBEE, U3 MB85RC64VPNF-G-JNERE1, U4 XC6220B331MR-G, U5 XC6220B331MR-G, U6 XC6220B331MR-G, Y1 Crystal

Commit message: Huellas actualizadas y lista de redes generada.
Parts:
- 0.1uF1, C1, C10, C12, C13, C14, C2, C3, C4, C5, C6, C7, C8, C9: footprint Capacitors_SMD:C_1206_HandSoldering -> Capacitors_SMD:C_0805_HandSoldering
- 4k1, 4k2, R1, R10, R11, R2, R3, R4, R5, R6, R7, R8, R9: footprint Resistors_SMD:R_1812_HandSoldering -> Resistors_SMD:R_0805_HandSoldering
- J2, J3: footprint Pin_Headers:Pin_Header_Straight_1x10_Pitch1.27mm -> Pin_Headers:Pin_Header_Straight_1x10_Pitch2.54mm
- U1: footprint TQFP64 -> Housings_QFP:TQFP-64_10x10mm_Pitch0.5mm
- U3: footprint SOIC127P600X175-8N -> Housings_SOIC:SOIC-8_3.9x4.9mm_Pitch1.27mm
- U4, U5, U6: footprint SOT95P300X145-5N -> sot:IC-SOT25
Changed lines of the file:
@@
 F 0 "R1" H 4130 7870 50  0000 L CNN
 F 1 "R_Small" H 4130 7810 50  0000 L CNN
-F 2 "Resistors_SMD:R_1812_HandSoldering" H 4100 7850 50  0001 C CNN
+F 2 "Resistors_SMD:R_0805_HandSoldering" H 4100 7850 50  0001 C CNN
 F 3 "" H 4100 7850 50  0001 C CNN
 	1    4100 7850
@@
 F 0 "U1" H 900 5200 50  0000 C CNN
 F 1 "SAMD20J18A-AU" H 4000 1900 50  0000 C CNN
-F 2 "TQFP64" H 2550 2400 50  0001 C CIN
+F 2 "Housings_QFP:TQFP-64_10x10mm_Pitch0.5mm" H 2550 2400 50  0001 C CIN
 F 3 "" H 2550 3800 50  0001 C CNN
 	1    2550 3550
@@
 F 0 "C4" H 2675 1650 50  0000 L CNN
 F 1 "C" H 2675 1450 50  0000 L CNN
-F 2 "Capacitors_SMD:C_1206_HandSoldering" H 2688 1400 50  0001 C CNN
+F 2 "Capacitors_SMD:C_0805_HandSoldering" H 2688 1400 50  0001 C CNN
 F 3 "" H 2650 1550 50  0001 C CNN
 	1    2650 1550
@@
 F 0 "C3" H 2675 1300 50  0000 L CNN
 F 1 "C" H 2675 1100 50  0000 L CNN
-F 2 "Capacitors_SMD:C_1206_HandSoldering" H 2688 1050 50  0001 C CNN
+F 2 "Capacitors_SMD:C_0805_HandSoldering" H 2688 1050 50  0001 C CNN
 F 3 "" H 2650 1200 50  0001 C CNN
 	1    2650 1200
@@
 F 0 "C2" H 2675 1100 50  0000 L CNN
 F 1 "C" H 2675 900 50  0000 L CNN
-F 2 "Capacitors_SMD:C_1206_HandSoldering" H 2688 850 50  0001 C CNN
+F 2 "Capacitors_SMD:C_0805_HandSoldering" H 2688 850 50  0001 C CNN
 F 3 "" H 2650 1000 50  0001 C CNN
 	1    2650 1000
@@
 F 0 "C1" H 2675 900 50  0000 L CNN
 F 1 "C" H 2675 700 50  0000 L CNN
-F 2 "Capacitors_SMD:C_1206_HandSoldering" H 2688 650 50  0001 C CNN
+F 2 "Capacitors_SMD:C_0805_HandSoldering" H 2688 650 50  0001 C CNN
 F 3 "" H 2650 800 50  0001 C CNN
 	1    2650 800
@@
 F 0 "C5" H 3275 1800 50  0000 L CNN
 F 1 "C" H 3275 1600 50  0000 L CNN
-F 2 "Capacitors_SMD:C_1206_HandSoldering" H 3288 1550 50  0001 C CNN
+F 2 "Capacitors_SMD:C_0805_HandSoldering" H 3288 1550 50  0001 C CNN
 F 3 "" H 3250 1700 50  0001 C CNN
 	1    3250 1700
@@
 F 0 "C6" H 4675 2050 50  0000 L CNN
 F 1 "C" H 4675 1850 50  0000 L CNN
-F 2 "Capacitors_SMD:C_1206_HandSoldering" H 4688 1800 50  0001 C CNN
+F 2 "Capacitors_SMD:C_0805_HandSoldering" H 4688 1800 50  0001 C CNN
 F 3 "" H 4650 1950 50  0001 C CNN
 	1    4650 1950
@@
 F 0 "C7" H 5075 2050 50  0000 L CNN
 F 1 "C" H 5075 1850 50  0000 L CNN
-F 2 "Capacitors_SMD:C_1206_HandSoldering" H 5088 1800 50  0001 C CNN
+F 2 "Capacitors_SMD:C_0805_HandSoldering" H 5088 1800 50  0001 C CNN
 F 3 "" H 5050 1950 50  0001 C CNN
 	1    5050 1950
@@
 F 0 "R2" V 5780 3300 50  0000 C CNN
 F 1 "R" V 5700 3300 50  0000 C CNN
-F 2 "Resistors_SMD:R_1812_HandSoldering" V 5630 3300 50  0001 C CNN
+F 2 "Resistors_SMD:R_0805_HandSoldering" V 5630 3300 50  0001 C CNN
 F 3 "" H 5700 3300 50  0001 C CNN
 	1    5700 3300
@@
 F 0 "R9" V 13180 1650 50  0000 C CNN
 F 1 "R" V 13100 1650 50  0000 C CNN
-F 2 "Resistors_SMD:R_1812_HandSoldering" V 13030 1650 50  0001 C CNN
+F 2 "Resistors_SMD:R_0805_HandSoldering" V 13030 1650 50  0001 C CNN
 F 3 "" H 13100 1650 50  0001 C CNN
 	1    13100 1650
@@
 F 0 "R6" V 9280 1150 50  0000 C CNN
 F 1 "R" V 9200 1150 50  0000 C CNN
-F 2 "Resistors_SMD:R_1812_HandSoldering" V 9130 1150 50  0001 C CNN
+F 2 "Resistors_SMD:R_0805_HandSoldering" V 9130 1150 50  0001 C CNN
 F 3 "" H 9200 1150 50  0001 C CNN
 	1    9200 1150
@@
 F 0 "R5" V 9030 1550 50  0000 C CNN
 F 1 "R" V 8950 1550 50  0000 C CNN
-F 2 "Resistors_SMD:R_1812_HandSoldering" V 8880 1550 50  0001 C CNN
+F 2 "Resistors_SMD:R_0805_HandSoldering" V 8880 1550 50  0001 C CNN
 F 3 "" H 8950 1550 50  0001 C CNN
 	1    8950 1550
@@
 F 0 "R3" H 7080 2720 50  0000 L CNN
 F 1 "R_Small" H 7080 2660 50  0000 L CNN
-F 2 "Resistors_SMD:R_1812_HandSoldering" H 7050 2700 50  0001 C CNN
+F 2 "Resistors_SMD:R_0805_HandSoldering" H 7050 2700 50  0001 C CNN
 F 3 "" H 7050 2700 50  0001 C CNN
 	1    7050 2700
@@
 F 0 "R4" H 7080 2820 50  0000 L CNN
 F 1 "R_Small" H 7080 2760 50  0000 L CNN
-F 2 "Resistors_SMD:R_1812_HandSoldering" H 7050 2800 50  0001 C CNN
+F 2 "Resistors_SMD:R_0805_HandSoldering" H 7050 2800 50  0001 C CNN
 F 3 "" H 7050 2800 50  0001 C CNN
 	1    7050 2800
@@
 F 0 "0.1uF1" H 10175 1400 50  0000 L CNN
 F 1 "C" H 10175 1200 50  0000 L CNN
-F 2 "Capacitors_SMD:C_1206_HandSoldering" H 10188 1150 50  0001 C CNN
+F 2 "Capacitors_SMD:C_0805_HandSoldering" H 10188 1150 50  0001 C CNN
 F 3 "" H 10150 1300 50  0001 C CNN
 	1    10150 1300
@@
 F 0 "U3" H 11251 1844 50  0000 L BNN
 F 1 "MB85RC64VPNF-G-JNERE1" H 11256 274 50  0000 L BNN
-F 2 "SOIC127P600X175-8N" H 11450 1250 50  0001 L BNN
+F 2 "Housings_SOIC:SOIC-8_3.9x4.9mm_Pitch1.27mm" H 11450 1250 50  0001 L BNN
 F 3 "SOP-8 Fujitsu" H 11450 1250 50  0001 L BNN
 F 4 "Bad" H 11450 1250 50  0001 L BNN "Campo4"
@@
 F 0 "4k1" V 5030 2900 50  0000 C CNN
 F 1 "R" V 4950 2900 50  0000 C CNN
-F 2 "Resistors_SMD:R_1812_HandSoldering" V 4880 2900 50  0001 C CNN
+F 2 "Resistors_SMD:R_0805_HandSoldering" V 4880 2900 50  0001 C CNN
 F 3 "" H 4950 2900 50  0001 C CNN
 	1    4950 2900
@@
 F 0 "4k2" V 5180 2900 50  0000 C CNN
 F 1 "R" V 5100 2900 50  0000 C CNN
-F 2 "Resistors_SMD:R_1812_HandSoldering" V 5030 2900 50  0001 C CNN
+F 2 "Resistors_SMD:R_0805_HandSoldering" V 5030 2900 50  0001 C CNN
 F 3 "" H 5100 2900 50  0001 C CNN
 	1    5100 2900
@@
 F 0 "C12" H 13675 3100 50  0000 L CNN
 F 1 "C" H 13675 2900 50  0000 L CNN
-F 2 "Capacitors_SMD:C_1206_HandSoldering" H 13688 2850 50  0001 C CNN
+F 2 "Capacitors_SMD:C_0805_HandSoldering" H 13688 2850 50  0001 C CNN
 F 3 "" H 13650 3000 50  0001 C CNN
 	1    13650 3000
@@
 F 0 "U5" H 14764 3009 50  0000 L CNN
 F 1 "XC6220B331MR-G" H 14727 2909 50  0000 L CNN
-F 2 "SOT95P300X145-5N" H 14950 2650 50  0001 L CNN
+F 2 "sot:IC-SOT25" H 14950 2650 50  0001 L CNN
 F 3 "XC6220 1A LDO655mV dropout 3.3Vout" H 15150 2050 50  0001 L CNN
 F 4 "MCP73831T-2ATI/OT" H 14950 2650 50  0001 L CNN "MP"
@@
 F 0 "R10" V 14180 2950 50  0000 C CNN
 F 1 "R" V 14100 2950 50  0000 C CNN
-F 2 "Resistors_SMD:R_1812_HandSoldering" V 14030 2950 50  0001 C CNN
+F 2 "Resistors_SMD:R_0805_HandSoldering" V 14030 2950 50  0001 C CNN
 F 3 "" H 14100 2950 50  0001 C CNN
 	1    14100 2950
@@
 F 0 "C14" H 14025 1450 50  0000 L CNN
 F 1 "C" H 14025 1250 50  0000 L CNN
-F 2 "Capacitors_SMD:C_1206_HandSoldering" H 14038 1200 50  0001 C CNN
+F 2 "Capacitors_SMD:C_0805_HandSoldering" H 14038 1200 50  0001 C CNN
 F 3 "" H 14000 1350 50  0001 C CNN
 	1    14000 1350
@@
 F 0 "U4" H 14764 1509 50  0000 L CNN
 F 1 "XC6220B331MR-G" H 14727 1409 50  0000 L CNN
-F 2 "SOT95P300X145-5N" H 14950 1150 50  0001 L CNN
+F 2 "sot:IC-SOT25" H 14950 1150 50  0001 L CNN
 F 3 "XC6220 1A LDO655mV dropout 3.3Vout" H 15150 550 50  0001 L CNN
 F 4 "MCP73831T-2ATI/OT" H 14950 1150 50  0001 L CNN "MP"
@@
 F 0 "C13" H 13675 4600 50  0000 L CNN
 F 1 "C" H 13675 4400 50  0000 L CNN
-F 2 "Capacitors_SMD:C_1206_HandSoldering" H 13688 4350 50  0001 C CNN
+F 2 "Capacitors_SMD:C_0805_HandSoldering" H 13688 4350 50  0001 C CNN
 F 3 "" H 13650 4500 50  0001 C CNN
 	1    13650 4500
@@
 F 0 "U6" H 14764 4509 50  0000 L CNN
 F 1 "XC6220B331MR-G" H 14727 4409 50  0000 L CNN
-F 2 "SOT95P300X145-5N" H 14950 4150 50  0001 L CNN
+F 2 "sot:IC-SOT25" H 14950 4150 50  0001 L CNN
 F 3 "XC6220 1A LDO655mV dropout 3.3Vout" H 15150 3550 50  0001 L CNN
 F 4 "MCP73831T-2ATI/OT" H 14950 4150 50  0001 L CNN "MP"
@@
 F 0 "R11" V 14180 4450 50  0000 C CNN
 F 1 "R" V 14100 4450 50  0000 C CNN
-F 2 "Resistors_SMD:R_1812_HandSoldering" V 14030 4450 50  0001 C CNN
+F 2 "Resistors_SMD:R_0805_HandSoldering" V 14030 4450 50  0001 C CNN
 F 3 "" H 14100 4450 50  0001 C CNN
 	1    14100 4450
@@
 F 0 "R7" V 9980 5200 50  0000 C CNN
 F 1 "330" V 9900 5200 50  0000 C CNN
-F 2 "Resistors_SMD:R_1812_HandSoldering" V 9830 5200 50  0001 C CNN
+F 2 "Resistors_SMD:R_0805_HandSoldering" V 9830 5200 50  0001 C CNN
 F 3 "" H 9900 5200 50  0001 C CNN
 	1    9900 5200
@@
 F 0 "R8" V 10330 4550 50  0000 C CNN
 F 1 "10k" V 10250 4550 50  0000 C CNN
-F 2 "Resistors_SMD:R_1812_HandSoldering" V 10180 4550 50  0001 C CNN
+F 2 "Resistors_SMD:R_0805_HandSoldering" V 10180 4550 50  0001 C CNN
 F 3 "" H 10250 4550 50  0001 C CNN
 	1    10250 4550
@@
 F 0 "C10" H 10525 5300 50  0000 L CNN
 F 1 "100nF" H 10525 5100 50  0000 L CNN
-F 2 "Capacitors_SMD:C_1206_HandSoldering" H 10538 5050 50  0001 C CNN
+F 2 "Capacitors_SMD:C_0805_HandSoldering" H 10538 5050 50  0001 C CNN
 F 3 "" H 10500 5200 50  0001 C CNN
 	1    10500 5200
@@
 F 0 "J2" H 7600 5450 50  0000 C CNN
 F 1 "Conn_01x10" H 7600 4350 50  0000 C CNN
-F 2 "Pin_Headers:Pin_Header_Straight_1x10_Pitch1.27mm" H 7600 4950 50  0001 C CNN
+F 2 "Pin_Headers:Pin_Header_Straight_1x10_Pitch2.54mm" H 7600 4950 50  0001 C CNN
 F 3 "" H 7600 4950 50  0001 C CNN
 	1    7600 4950
@@
 F 0 "J3" H 8000 5550 50  0000 C CNN
 F 1 "Conn_01x10" H 8000 4450 50  0000 C CNN
-F 2 "Pin_Headers:Pin_Header_Straight_1x10_Pitch1.27mm" H 8000 5050 50  0001 C CNN
+F 2 "Pin_Headers:Pin_Header_Straight_1x10_Pitch2.54mm" H 8000 5050 50  0001 C CNN
 F 3 "" H 8000 5050 50  0001 C CNN
 	1    8000 5050
@@
 F 0 "C8" H 10075 3050 50  0000 L CNN
 F 1 "1uf" H 10075 2850 50  0000 L CNN
-F 2 "Capacitors_SMD:C_1206_HandSoldering" H 10088 2800 50  0001 C CNN
+F 2 "Capacitors_SMD:C_0805_HandSoldering" H 10088 2800 50  0001 C CNN
 F 3 "" H 10050 2950 50  0001 C CNN
 	1    10050 2950
@@
 F 0 "C9" H 10375 3050 50  0000 L CNN
 F 1 "100nf" H 10375 2850 50  0000 L CNN
-F 2 "Capacitors_SMD:C_1206_HandSoldering" H 10388 2800 50  0001 C CNN
+F 2 "Capacitors_SMD:C_0805_HandSoldering" H 10388 2800 50  0001 C CNN
 F 3 "" H 10350 2950 50  0001 C CNN
 	1    10350 2950
